File: CALCAGAINFINALFINALFINAL/kicad-files/esp32-s3-pinout.kicad_sch (KiCad schematic)
At the start: 13 parts, among them J3 Micro_SD_Card, U8 ESP32-S3-WROOM-1

Commit message: Turns out my whole power thing was absolutely retarded i should REALLY stop relying on gemini its actually retarded as fuh. Ima start js rawdogging it w forums and reddit. once its functional ima order it. i gota remember there no deadline better do it right the first time.
Parts:
- C1: LCSC C1525 -> C1848
- R1, R2, R3: footprint Resistor_SMD:R_0201_0603Metric -> Resistor_SMD:R_0603_1608Metric
- U8: value ESP32-S3-WROOM-1 -> ESP32-S3-WROOM-2; footprint RF_Module:ESP32-S3-WROOM-1 -> RF_Module:ESP32-S3-WROOM-2; now left out of the parts list
Connections:
- net en is gone; now on net 3V3: U8.3 (EN)
- net ~{INT1} is gone; now on net OV_HREF: U8.9 (IO16)
- net OV_HREF: no longer U8.35 (IO42)
- net boot: now reaches R6.2, U8.27 (IO0)
- net batprog: now reaches U8.24 (IO47)
- new net BL: U8.35 (IO42)
Changed lines of the file:
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@@
+		)
+	)
+	(label "boot"
+		(at 191.008 118.872 0)
+		(effects
+			(font
+				(size 1.27 1.27)
+			)
+			(justify left bottom)
 		)
 	)
@@
 		)
 	)
-	(label "OV_HREF"
+	(label "BL"
 		(at 160.528 88.392 180)
 		(effects
@@
 		)
 	)
-	(label "~{INT1}"
+	(label "OV_HREF"
 		(at 191.008 78.232 0)
 		(effects
@@
 			)
 			(justify right top)
+		)
+	)
+	(label "batprog"
+		(at 160.528 80.772 180)
+		(effects
+			(font
+				(size 1.27 1.27)
+			)
+			(justify right bottom)
 		)
 	)
@@
 		)
 	)
-	(global_label "VCC"
+	(global_label "en"
 		(shape input)
 		(at 98.806 42.926 0)
@@
 			)
 		)
-		(property "Footprint" "Resistor_SMD:R_0201_0603Metric"
+		(property "Footprint" "Resistor_SMD:R_0603_1608Metric"
 			(at 77.724 47.244 90)
 			(hide yes)
@@
 			)
 		)
-		(property "Description" "Resistor"
+		(property "Description" ""
 			(at 77.724 45.466 0)
 			(hide yes)
@@
 		(body_style 1)
 		(exclude_from_sim no)
-		(in_bom yes)
+		(in_bom no)
 		(on_board yes)
 		(in_pos_files yes)
@@
 			)
 		)
-		(property "Value" "ESP32-S3-WROOM-1"
+		(property "Value" "ESP32-S3-WROOM-2"
 			(at 178.8861 73.152 0)
 			(show_name no)
@@
 			)
 		)
-		(property "Footprint" "RF_Module:ESP32-S3-WROOM-1"
+		(property "Footprint" "RF_Module:ESP32-S3-WROOM-2"
 			(at 175.768 103.632 0)
 			(hide yes)
@@
 			)
 		)
-		(property "Datasheet" "https://www.espressif.com/sites/default/files/documentation/esp32-s3-wroom-1_wroom-1u_datasheet_en.pdf"
+		(property "Datasheet" ""
 			(at 175.768 101.092 0)
 			(hide yes)
@@
 			)
 		)
-		(property "Description" "RF Module, ESP32-S3 SoC, Wi-Fi 802.11b/g/n, Bluetooth, BLE, 32-bit, 3.3V, onboard antenna, SMD"
+		(property "Description" ""
 			(at 175.768 101.092 0)
 			(hide yes)
@@
 					(variant
 						(name "goody2shoes-nocamera")
+						(in_bom yes)
 					)
 				)
@@
 			)
 		)
-		(property "LCSC" "C1525"
+		(property "LCSC" "C1848"
 			(at 90.424 39.116 0)
 			(hide yes)
@@
 			)
 		)
-		(property "Footprint" "Resistor_SMD:R_0201_0603Metric"
+		(property "Footprint" "Resistor_SMD:R_0603_1608Metric"
 			(at 77.724 37.084 90)
 			(hide yes)
@@
 			)
 		)
-		(property "Description" "Resistor"
+		(property "Description" ""
 			(at 77.724 35.306 0)
 			(hide yes)
@@
 			)
 		)
-		(property "Datasheet" "https://www.we-online.com/components/products/datasheet/693072010801.pdf"
+		(property "Datasheet" ""
 			(at 46.99 42.926 0)
 			(hide yes)
@@
 			)
 		)
-		(property "Description" "Micro SD Card Socket"
+		(property "Description" ""
 			(at 46.99 42.926 0)
 			(hide yes)
@@
 			)
 		)
-		(property "Footprint" "Resistor_SMD:R_0201_0603Metric"
+		(property "Footprint" "Resistor_SMD:R_0603_1608Metric"
 			(at 77.724 49.784 90)
 			(hide yes)
@@
 			)
 		)
-		(property "Description" "Resistor"
+		(property "Description" ""
 			(at 77.724 48.006 0)
 			(hide yes)
