File: CALCAGAINFINALFINALFINAL/kicad-files/esp32-s3-pinout.kicad_sch (KiCad schematic)
At the start: 13 parts, among them J3 Micro_SD_Card, U8 ESP32-S3-WROOM-2

Commit message: workin on matching up the pcb with the schematic gona chuck it on pcbreview then wait till i can stack up enough cash to order the first pcba. i need to make sure the design is 100% otherwise im js spending 300 bucks on a paperweight. so far the logic seems good js need to fix up some clerical errors w schematic.
Parts:
- removed H1, H2, H3, H4, H5: MountingHole_Pad, MountingHole:MountingHole_2.5mm_Pad, symbol Mechanical:MountingHole_Pad
- added J1: Conn_01x40, symbol Connector_Generic:Conn_01x40
- added R13: 10k, symbol Device:R
- added R7: 1k, symbol Device:R
- added U1: 74AUC2G08, Package_TO_SOT_SMD:SOT-223-5, symbol 74xGxx:74AUC2G08
- J3: footprint Connector_Card:microSD_HC_Molex_47219-2001 -> ButtonPads:CONN_47219-2001_MOL
- R1, R3: value R -> 10k
- U8: LCSC (none) -> C2913202; now in the parts list
Connections:
- net 3V3: now also J1.12 (Pin_12), J1.39 (Pin_39), J1.6 (Pin_6), J1.7 (Pin_7); no longer C1.1, C2.1, J3.4 (VDD), U8.3 (EN)
- net BL: now also R13.2, R7.2, U1.7
- net GND: now also J1.16 (Pin_16), J1.37 (Pin_37), J1.38 (Pin_38), J1.40 (Pin_40), J1.5 (Pin_5), U1.1
- net MOSI: now also J1.13 (Pin_13)
- net RST: now also J1.15 (Pin_15)
- net SDA: now also U8.24 (IO47); no longer U8.7 (IO7)
- net batprog: now also U8.7 (IO7); no longer U8.24 (IO47)
- new net 2.8V: J1.33 (Pin_33)
- new net cathode: J1.34 (Pin_34), J1.35 (Pin_35), J1.36 (Pin_36), U1.2
- new net en: C1.1, C2.1, J3.4 (VDD), U8.3 (EN)
- no-connect marks 2 -> 36
Other:
- note added: "Binary backlight control logic AND"
- note added: "TODO: 1. update schematic to match pcb 2.run erc to make sure its all alright"
- note added: "display 40pin fpc connector"
- note removed: "Display pins"

Commit message: yo chat this actually for reals the order now im ordering it and neva openin kicad again ong
Parts:
- added C3: 10uf, Capacitor_SMD:C_0603_1608Metric, symbol Device:C
- added R14: 10k, symbol Device:R
- added REF**1: PinHeader_2x09_P2.54mm_Vertical, symbol Connector_Generic:Conn_02x09_Top_Bottom
- added SW1, SW2: SW_DPST_x2, symbol Switch:SW_DPST_x2
- added U1: TPS73125DBV, Package_TO_SOT_SMD:SOT-23-5, symbol Regulator_Linear:TPS73125DBV
- R7: value 1k -> 1.25
- S1: renamed from J1; value Conn_01x40 -> Omron_XF2M-4015-1A_1x40-1MP_P0.5mm_Horizontal
- SOt-23: renamed from U1; value 74AUC2G08 -> idk; footprint Package_TO_SOT_SMD:SOT-223-5 -> Package_TO_SOT_SMD:SOT-23; symbol 74xGxx:74AUC2G08 -> Transistor_FET:2N7002
Connections:
- net 3V3: now also R6.1, C3.1, R14.2, REF**1.2 (Pin_2), REF**1.8 (Pin_8), SW2.2 (B), U1.1 (IN), U1.3 (EN), U1.4 (NR); no longer S1.39 (Pin_39)
- net BL: now also SOt-23.1 (G); no longer R7.2, SOt-23.7
- net CS: now also S1.9 (Pin_9)
- net DC: now also S1.10 (Pin_10)
- net GND: now also R13.1, SOt-23.2 (S), C3.2, REF**1.1 (Pin_1), REF**1.17 (Pin_17), SW1.1 (A), SW2.1 (A), U1.2 (GND); no longer R6.1, SOt-23.1
- net OV_D0: now also REF**1.7 (Pin_7)
- net OV_D1: now also REF**1.9 (Pin_9)
- net OV_D2: now also REF**1.10 (Pin_10)
- net OV_D3: now also REF**1.11 (Pin_11)
- net OV_D4: now also REF**1.12 (Pin_12)
- net OV_D5: now also REF**1.13 (Pin_13)
- net OV_D6: now also REF**1.14 (Pin_14)
- net OV_D7: now also REF**1.16 (Pin_16)
- net OV_HREF: now also REF**1.6 (Pin_6)
- net OV_PCLK: now also REF**1.15 (Pin_15)
- net OV_VSYNC: now also REF**1.4 (Pin_4)
- net SCK: now also S1.11 (Pin_11)
- net SCL: now also REF**1.3 (Pin_3)
- net SDA: now also REF**1.5 (Pin_5)
- net boot: now also SW1.2 (B)
- net cathode: now also SOt-23.3 (D); no longer SOt-23.2
- net en: now also R14.1; no longer C1.1, C2.1, J3.4 (VDD)
- net 2V8: now reaches R7.1
- net 2V8: now also S1.39 (Pin_39), U1.5 (OUT)
- net 2.8V: no longer names the net of S1.33 (Pin_33)
- net 2.8V: now also R7.2
- new net: C1.1, C2.1, J3.4 (VDD)
- no-connect marks 36 -> 34
Other:
- moved on the sheet: R13, U8
