File: CALCAGAINFINALFINALFINAL/kicad-files/.portability/backup/Cfx-port.kicad_pcb (KiCad board)
At the start: 4 copper layers, 65 x 135.9 mm, 98 parts, among them J2 USB_C_Receptacle_USB2.0_16P, J3 Micro_SD_Card, J4 Conn_01x02, Q1 DMP3099L, SW100 SW_SPST, SW101 SW_SPST, SW49 SW_SPST, SW52 SW_SPST, SW55 SW_SPST, SW56 SW_SPST, SW57 SW_SPST, SW58 SW_SPST, SW59 SW_SPST, SW60 SW_SPST, SW61 SW_SPST, SW62 SW_SPST, SW63 SW_SPST, SW64 SW_SPST, SW65 SW_SPST, SW66 SW_SPST, SW67 SW_SPST, SW68 SW_SPST, SW69 SW_SPST, SW70 SW_SPST, SW71 SW_SPST, SW72 SW_SPST, SW73 SW_SPST, SW74 SW_SPST, SW75 SW_SPST, SW76 SW_SPST, SW77 SW_SPST, SW78 SW_SPST, SW79 SW_SPST, SW80 SW_SPST, SW81 SW_SPST, SW82 SW_SPST, SW83 SW_SPST, SW84 SW_SPST, SW85 SW_SPST, SW86 SW_SPST, SW87 SW_SPST, SW88 SW_SPST, SW89 SW_SPST, SW90 SW_SPST, SW91 SW_SPST, SW92 SW_SPST, SW93 SW_SPST, SW94 SW_SPST, SW95 SW_SPST, SW96 SW_SPST, SW97 SW_SPST, SW98 SW_SPST, SW99 SW_SPST, U5 TP4056-42-ESOP8, U7 TCA9535DBR, U8 ESP32-S3-WROOM-2

Commit message: there were some errrors in the initial order but its all good now. should come here in 2 weeks.
Parts:
- removed the SOt-23 at (102.1, 66.0)
- removed r11, r18: 10k, Resistor_SMD:R_0603_1608Metric
- added 23s: 1k, Resistor_SMD:R_0603_1608Metric_Pad0.98x0.95mm_HandSolder, B.Cu at (117.6, 53.5)
- added 3a: 1k, Resistor_SMD:R_0603_1608Metric_Pad0.98x0.95mm_HandSolder, B.Cu at (121.4, 52.3)
- added C1: 0.1, Capacitor_SMD:C_0603_1608Metric, B.Cu at (101.5, 64.2)
- added R5: 4.7k, Resistor_SMD:R_0603_1608Metric, B.Cu at (132.3, 43.6)
- added REE: 1k, Resistor_SMD:R_0603_1608Metric_Pad0.98x0.95mm_HandSolder, B.Cu at (107.7, 50.2)
- added U1: TPS73125DBV, Package_TO_SOT_SMD:SOT-23-5, B.Cu at (102.3, 69.1)
- added f23: 1k, Resistor_SMD:R_0603_1608Metric_Pad0.98x0.95mm_HandSolder, B.Cu at (109.7, 51.3)
- added r213: 1k, Resistor_SMD:R_0603_1608Metric_Pad0.98x0.95mm_HandSolder, B.Cu at (111.4, 55.9)
- added r231: 1k, Resistor_SMD:R_0603_1608Metric_Pad0.98x0.95mm_HandSolder, B.Cu at (107.7, 54.5)
- added r233: 1k, Resistor_SMD:R_0603_1608Metric_Pad0.98x0.95mm_HandSolder, B.Cu at (114.6, 56.9)
- added re1: 1k, Resistor_SMD:R_0603_1608Metric_Pad0.98x0.95mm_HandSolder, B.Cu at (121.4, 54.9)
- added v23: 1k, Resistor_SMD:R_0603_1608Metric_Pad0.98x0.95mm_HandSolder, B.Cu at (117.6, 51.2)
- added we2: 1k, Resistor_SMD:R_0603_1608Metric_Pad0.98x0.95mm_HandSolder, B.Cu at (117.6, 55.9)
- D1: value D_SOD-123 -> D_0201_0603Metric; footprint Diode_SMD:D_SOD-123 -> Diode_SMD:D_0201_0603Metric
- D15: renamed from D6; footprint Diode_SMD:D_0603_1608Metric -> LED_SMD:LED_01005_0402Metric
- D15: renamed from D5; footprint Diode_SMD:D_0603_1608Metric -> LED_SMD:LED_01005_0402Metric
- D3: renamed from D2; value D_SOD-123 -> D_0201_0603Metric; footprint Diode_SMD:D_SOD-123 -> Diode_SMD:D_0201_0603Metric
- D6: renamed from D3; value D_SOD-123 -> D_0201_0603Metric; footprint Diode_SMD:D_SOD-123 -> Diode_SMD:D_0201_0603Metric
- J2: footprint Connector_USB:USB_C_Receptacle_GCT_USB4105-xx-A_16P_TopMnt_Horizontal -> ButtonPads:TENSILITY_54-00304
- J4: footprint Connector_JST:JST_PH_S2B-PH-K_1x02_P2.00mm_Horizontal -> Connector_JST:JST_XH_S2B-XH-A-1_1x02_P2.50mm_Horizontal
- R12: value 1.2 -> 1.6
- R67: renamed from R17; value 510 -> 1k
- S1: value CONN40_AFC01-S40FCA-00_JUS -> Omron_XF2M-4015-1A_1x40-1MP_P0.5mm_Horizontal; footprint ButtonPads:CONN40_AFC01-S40FCA-00_JUS -> Connector_FFC-FPC:Omron_XF2M-4015-1A_1x40-1MP_P0.5mm_Horizontal
- moved cuba 15.5 mm to (145.5, 107.2)
- moved r21 12.0 mm to (142.2, 106.5), turned to 180 degrees
- moved D1 7.40 mm to (103.3, 74.0), turned to 180 degrees
- moved R9 5.46 mm to (153.3, 115.9), turned to -90 degrees
- moved toes4 4.75 mm to (125.7, 48.8)
- moved J2 4.63 mm to (160.9, 112.7)
- moved C6 3.03 mm to (129.4, 93.9), turned to 90 degrees
- moved R8 2.81 mm to (153.2, 108.3)
- moved toes1 2.40 mm to (129.0, 41.6), turned to 180 degrees
- moved D15 2.06 mm to (146.6, 85.6)
- moved C2 1.83 mm to (101.5, 62.0), turned to 180 degrees
- moved D15 1.66 mm to (146.8, 87.3)
- moved R3 1.20 mm to (131.4, 30.3), turned to 90 degrees
- moved NIGERC 1.01 mm to (140.4, 103.7), turned to 90 degrees
- moved SW99 0.95 mm to (158.7, 83.8)
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- renumbered C3 to C5, C5 to C6, C4 to C6, D4 to D8, r15 to NIGERC, R10 to R1, R1 to R10, R2 to R11, R6 to R123, R9 to R2, r13 to R3, R7 to R5, r12 to R55, r11 to R67, r19 to R8, R3 to R9, R8 to R902, r14 to cuba, r16 to r21, r4 to r2123, d7 to toes1, d8 to toes4
Connections:
- S1 pad 10: /esp32-s3 pinout/SCK -> /esp32-s3 pinout/DC
- S1 pad 11: /esp32-s3 pinout/DC -> /esp32-s3 pinout/SCK
- S1 pad 17: GND -> unconnected-(S1-Pin_17-Pad17)
- S1 pad 18: GND -> unconnected-(S1-Pin_18-Pad18)
- S1 pad 19: GND -> unconnected-(S1-Pin_19-Pad19)
- S1 pad 20: GND -> unconnected-(S1-Pin_20-Pad20)
- S1 pad 21: GND -> unconnected-(S1-Pin_21-Pad21)
- S1 pad 22: GND -> unconnected-(S1-Pin_22-Pad22)
- S1 pad 23: GND -> unconnected-(S1-Pin_23-Pad23)
- S1 pad 24: GND -> unconnected-(S1-Pin_24-Pad24)
- S1 pad 25: GND -> unconnected-(S1-Pin_25-Pad25)
- S1 pad 26: GND -> unconnected-(S1-Pin_26-Pad26)
- S1 pad 27: GND -> unconnected-(S1-Pin_27-Pad27)
- S1 pad 28: GND -> unconnected-(S1-Pin_28-Pad28)
- S1 pad 29: GND -> unconnected-(S1-Pin_29-Pad29)
- S1 pad 30: GND -> unconnected-(S1-Pin_30-Pad30)
- S1 pad 31: GND -> unconnected-(S1-Pin_31-Pad31)
- S1 pad 32: GND -> unconnected-(S1-Pin_32-Pad32)
- U8 pad 25: 2v8ce -> unconnected-(U8-IO48-Pad25)
Routing:
- net 2v8ce: track 72.1 -> 0.00 mm, vias 2 -> 0
- net batprog: track 99.1 -> 61.1 mm, vias 2 -> 4
- net VCC: track 77.6 -> 94.3 mm, vias 0 -> 2
- net /Keypad Matrix/R1: track 125.1 -> 133.8 mm
- net /power-ic/BAT+: track 83.2 -> 75.1 mm
- net 3V3: track 190.0 -> 197.4 mm, vias 5 -> 7
- net usb_N: track 76.6 -> 83.7 mm, vias 2 -> 3
- net SDA: track 48.6 -> 42.6 mm, vias 3 -> 2
- net MOSI: track 38.6 -> 34.5 mm
- net /Keypad Matrix/R2: track 164.5 -> 160.5 mm, vias 8 -> 9
- net usb_P: track 76.4 -> 80.0 mm, vias 2 -> 5
- net 2V8: track 43.0 -> 39.6 mm
- net /Keypad Matrix/C5: track 133.4 -> 136.3 mm
- net BL: track 44.3 -> 41.9 mm
- net OV_VSYNC: track 33.2 -> 31.2 mm
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Other:
- board text added: "d"
- board text removed: "1"
