File: hardware/CALCAGAINFINALFINALFINAL/kicad-files/Cfx-port.kicad_pcb (KiCad board)
At the start: 4 copper layers, 65 x 135.9 mm, 98 parts, among them J2 USB_C_Receptacle_USB2.0_16P, J3 Micro_SD_Card, J4 Conn_01x02, Q1 DMP3099L, SW100 SW_SPST, SW101 SW_SPST, SW49 SW_SPST, SW52 SW_SPST, SW55 SW_SPST, SW56 SW_SPST, SW57 SW_SPST, SW58 SW_SPST, SW59 SW_SPST, SW60 SW_SPST, SW61 SW_SPST, SW62 SW_SPST, SW63 SW_SPST, SW64 SW_SPST, SW65 SW_SPST, SW66 SW_SPST, SW67 SW_SPST, SW68 SW_SPST, SW69 SW_SPST, SW70 SW_SPST, SW71 SW_SPST, SW72 SW_SPST, SW73 SW_SPST, SW74 SW_SPST, SW75 SW_SPST, SW76 SW_SPST, SW77 SW_SPST, SW78 SW_SPST, SW79 SW_SPST, SW80 SW_SPST, SW81 SW_SPST, SW82 SW_SPST, SW83 SW_SPST, SW84 SW_SPST, SW85 SW_SPST, SW86 SW_SPST, SW87 SW_SPST, SW88 SW_SPST, SW89 SW_SPST, SW90 SW_SPST, SW91 SW_SPST, SW92 SW_SPST, SW93 SW_SPST, SW94 SW_SPST, SW95 SW_SPST, SW96 SW_SPST, SW97 SW_SPST, SW98 SW_SPST, SW99 SW_SPST, U5 TP4056-42-ESOP8, U7 TCA9535DBR, U8 ESP32-S3-WROOM-2

Commit message: workin on v2
Parts:
- removed J3: Micro_SD_Card, ButtonPads:CONN_TF-01A_HRO
- removed the REF** at (129.2, 43.5)
- removed the SOt-23 at (102.1, 66.0)
- removed d8: 10uf, Capacitor_SMD:C_0603_1608Metric_Pad1.08x0.95mm_HandSolder
- removed the r11 at (105.3, 68.6)
- added REF**: NetTie-2_SMD_Pad0.5mm, NetTie:NetTie-2_SMD_Pad0.5mm, B.Cu at (101.0, 65.8)
- added REF**: R_0603_1608Metric_Pad0.98x0.95mm_HandSolder, Resistor_SMD:R_0603_1608Metric_Pad0.98x0.95mm_HandSolder, B.Cu at (108.0, 40.0)
- moved r11 6.84 mm to (117.2, 29.2)
- moved R17 4.40 mm to (111.8, 29.2)
- moved SOt-23 1.69 mm to (111.8, 37.7), turned to 0 degrees
Connections:
- SOt-23 pad 1: BL1 -> /esp32-s3 pinout/cathode
- SOt-23 pad 3: /esp32-s3 pinout/cathode -> BL1
Routing:
- net 2v8ce: track 72.1 -> 0.00 mm, vias 2 -> 0
- net OV_D7: track 43.9 -> 0.00 mm, vias 2 -> 0
- net OV_PCLK: track 41.3 -> 0.00 mm, vias 1 -> 0
- net OV_D5: track 41.1 -> 0.00 mm, vias 1 -> 0
- net OV_D0: track 41.1 -> 0.00 mm, vias 1 -> 0
- net OV_D1: track 40.4 -> 0.00 mm, vias 1 -> 0
- net OV_D6: track 35.7 -> 0.00 mm, vias 1 -> 0
- net OV_D3: track 35.3 -> 0.00 mm, vias 1 -> 0
- net OV_VSYNC: track 33.2 -> 0.00 mm, vias 1 -> 0
- net OV_HREF: track 28.2 -> 0.00 mm, vias 1 -> 0
- net 3V3: track 190.0 -> 167.4 mm, vias 5 -> 4
- net OV_D4: track 21.1 -> 0.00 mm, vias 2 -> 0
- net /esp32-s3 pinout/MISO: track 26.6 -> 9.02 mm
- net /esp32-s3 pinout/SCK: track 74.4 -> 60.7 mm, vias 4 -> 2
- net /esp32-s3 pinout/CMD: track 37.0 -> 25.9 mm, vias 4 -> 2
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Other:
- board text added: "TODO 0. [x] remove camera 1. [x] fix screen 2. [] fix battery 3. [] add sd card again"
- board text added: "backlight control shi"
